File: GPIO print/GPIO print.kicad_pcb (KiCad board)
At the start: 2 copper layers, 100 x 22 mm, 8 parts, among them J1 Raspberry Out, J2 Raspberry In, SW1 Power Switch

Commit message: Started sketch back panel
Parts:
- added REF**: OSHW-Logo2_7.3x6mm_SilkScreen, Symbol:OSHW-Logo2_7.3x6mm_SilkScreen, B.Cu at (176.2, 96.5)
Other:
- board text added: "GPIO Export Revision: 1"
